Commit message: fix: partial fix for robot xacro and attempted fix to nav2 stack

File: robot_description/mobile_manipulator/urdf/mobile_manipulator.urdf.xacro (robot description, xacro)
@@ -13,5 +13,5 @@
   <xacro:open_manipulator_x_gazebo prefix=""/>
   <!-- Mount arm to tower_sensor_plate with vertical offset and slight backward position -->
-  <!-- tower_sensor_plate is ~0.283m from base_link, add 0.04m clearance to avoid clipping -->
+  <!-- tower_sensor_plate is ~0.283m from base_link, add 0.02m clearance -->
   <!-- Position slightly backward (-0.02m X) to improve weight distribution and reduce forward tilt -->
   <!-- Rotate arm by -90° around Y-axis (pitch) to make it point upward instead of forward -->
@@ -20,5 +20,5 @@
     <parent link="tower_sensor_plate"/>
     <child link="link1"/>
-    <origin xyz="-0.02 0.0 0.04" rpy="0 ${arm_pitch} 0"/>
+    <origin xyz="-0.02 0.0 0.02" rpy="0 ${arm_pitch} 0"/>
   </joint>
   <!-- Counterweight to balance arm weight and prevent forward tilt -->

Commit message: fix: rviz issues (and migrate to turtlebot3)

File: robot_description/mobile_manipulator/urdf/mobile_manipulator.urdf.xacro (robot description, xacro)
@@ -3,6 +3,6 @@
   <!-- Define package path property -->
   <xacro:property name="mobile_manipulator_path" value="$(find mobile_manipulator)"/>
-  <!-- Include TurtleBot4 base -->
-  <xacro:include filename="$(find turtlebot4_description)/urdf/standard/turtlebot4.urdf.xacro"/>
+  <!-- Include TurtleBot3 Waffle base -->
+  <xacro:include filename="$(find turtlebot3_gazebo)/urdf/turtlebot3_waffle.urdf"/>
   <!-- Include official OpenManipulator-X arm -->
   <xacro:include filename="$(find open_manipulator_description)/urdf/open_manipulator_x/open_manipulator_x_arm.urdf.xacro"/>
@@ -12,46 +12,119 @@
   <!-- Instantiate Gazebo properties for arm -->
   <xacro:open_manipulator_x_gazebo prefix=""/>
-  <!-- Mount arm to tower_sensor_plate with vertical offset and slight backward position -->
-  <!-- tower_sensor_plate is ~0.283m from base_link, add 0.02m clearance -->
-  <!-- Position slightly backward (-0.02m X) to improve weight distribution and reduce forward tilt -->
+  <!-- Mount arm on top of the LIDAR scanner (base_scan link) -->
+  <!-- base_scan is at (-0.064, 0, 0.122) from base_link -->
+  <!-- Add small vertical offset to clear the LIDAR sensor -->
   <!-- Rotate arm by -90° around Y-axis (pitch) to make it point upward instead of forward -->
   <xacro:property name="arm_pitch" value="${-pi/2}"/>
   <joint name="arm_mount_joint" type="fixed">
-    <parent link="tower_sensor_plate"/>
+    <parent link="base_scan"/>
     <child link="link1"/>
-    <origin xyz="-0.02 0.0 0.02" rpy="0 ${arm_pitch} 0"/>
+    <origin xyz="0.0 0.0 0.04" rpy="0 ${arm_pitch} 0"/>
   </joint>
-  <!-- Counterweight to balance arm weight and prevent forward tilt -->
-  <!-- Positioned at center bottom of sensor tower, directly below the arm -->
-  <link name="counterweight_link">
-    <visual>
-      <origin xyz="0 0 0" rpy="0 0 0"/>
-      <geometry>
-        <cylinder radius="0.08" length="0.03"/>
-      </geometry>
-      <material name="counterweight_grey">
-        <color rgba="0.2 0.2 0.2 1.0"/>
-      </material>
-    </visual>
-    <collision>
-      <origin xyz="0 0 0" rpy="0 0 0"/>
-      <geometry>
-        <cylinder radius="0.08" length="0.03"/>
-      </geometry>
-    </collision>
-    <inertial>
-      <origin xyz="0 0 0" rpy="0 0 0"/>
-      <mass value="1.2"/>
-      <inertia ixx="0.003" ixy="0" ixz="0" iyy="0.003" iyz="0" izz="0.005"/>
-    </inertial>
-  </link>
-  <joint name="counterweight_joint" type="fixed">
-    <parent link="base_link"/>
-    <child link="counterweight_link"/>
-    <origin xyz="0.0 0.0 0.015" rpy="0 0 0"/>
-  </joint>
-  <!-- Gazebo material for counterweight -->
-  <gazebo reference="counterweight_link">
-    <material>Gazebo/Black</material>
+  <!-- Gazebo plugins for TurtleBot3 sensors and mobility (Gazebo Harmonic / gz-sim) -->
+  <!-- LIDAR sensor plugin using GPU LIDAR (Gazebo Harmonic compatible) -->
+  <gazebo reference="base_scan">
+    <sensor name="lidar" type="gpu_lidar">
+      <topic>scan</topic>
+      <update_rate>5</update_rate>
+      <gz_frame_id>base_scan</gz_frame_id>
+      <lidar>
+        <scan>
+          <horizontal>
+            <samples>360</samples>
+            <resolution>1</resolution>
+            <min_angle>0.0</min_angle>
+            <max_angle>6.28319</max_angle>
+          </horizontal>
+        </scan>
+        <range>
+          <min>0.12</min>
+          <max>3.5</max>
+          <resolution>0.015</resolution>
+        </range>
+        <noise>
+          <type>gaussian</type>
+          <mean>0.0</mean>
+          <stddev>0.01</stddev>
+        </noise>
+      </lidar>
+      <always_on>1</always_on>
+      <visualize>true</visualize>
+    </sensor>
+  </gazebo>
+  <!-- IMU sensor plugin (Gazebo Harmonic compatible) -->
+  <gazebo reference="imu_link">
+    <sensor name="imu_sensor" type="imu">
+      <topic>imu</topic>
+      <update_rate>200</update_rate>
+      <gz_frame_id>imu_link</gz_frame_id>
+      <always_on>1</always_on>
+      <visualize>true</visualize>
+      <imu>
+        <angular_velocity>
+          <x>
+            <noise type="gaussian">
+              <mean>0.0</mean>
+              <stddev>2e-4</stddev>
+            </noise>
+          </x>
+          <y>
+            <noise type="gaussian">
+              <mean>0.0</mean>
+              <stddev>2e-4</stddev>
+            </noise>
+          </y>
+          <z>
+            <noise type="gaussian">
+              <mean>0.0</mean>
+              <stddev>2e-4</stddev>
+            </noise>
+          </z>
+        </angular_velocity>
+        <linear_acceleration>
+          <x>
+            <noise type="gaussian">
+              <mean>0.0</mean>
+              <stddev>1.7e-2</stddev>
+            </noise>
+          </x>
+          <y>
+            <noise type="gaussian">
+              <mean>0.0</mean>
+              <stddev>1.7e-2</stddev>
+            </noise>
+          </y>
+          <z>
+            <noise type="gaussian">
+              <mean>0.0</mean>
+              <stddev>1.7e-2</stddev>
+            </noise>
+          </z>
+        </linear_acceleration>
+      </imu>
+    </sensor>
+  </gazebo>
+  <!-- Differential drive plugin for mobile base (Gazebo Harmonic compatible) -->
+  <gazebo>
+    <plugin filename="gz-sim-diff-drive-system" name="gz::sim::systems::DiffDrive">
+      <left_joint>wheel_left_joint</left_joint>
+      <right_joint>wheel_right_joint</right_joint>
+      <wheel_separation>0.287</wheel_separation>
+      <wheel_radius>0.033</wheel_radius>
+      <odom_publish_frequency>30</odom_publish_frequency>
+      <max_linear_acceleration>1.0</max_linear_acceleration>
+      <min_linear_acceleration>-1.0</min_linear_acceleration>
+      <max_angular_acceleration>2.0</max_angular_acceleration>
+      <min_angular_acceleration>-2.0</min_angular_acceleration>
+      <max_linear_velocity>0.26</max_linear_velocity>
+      <min_linear_velocity>-0.26</min_linear_velocity>
+      <max_angular_velocity>1.82</max_angular_velocity>
+      <min_angular_velocity>-1.82</min_angular_velocity>
+      <topic>cmd_vel</topic>
+      <odom_topic>/model/mobile_manipulator/odometry</odom_topic>
+      <tf_topic>/model/mobile_manipulator/tf</tf_topic>
+      <frame_id>odom</frame_id>
+      <child_frame_id>base_footprint</child_frame_id>
+    </plugin>
   </gazebo>
   <!-- Include ros2_control -->
