Commit message: fix: approach logic fix

File: robot_description/turtlebot3_manipulation_description/urdf/turtlebot3_manipulation.urdf.xacro (robot description, xacro)
@@ -28,4 +28,43 @@
   <xacro:open_manipulator_x prefix="$(arg prefix)" />
   <xacro:open_manipulator_x_gazebo prefix="$(arg prefix)" />
+  <!-- Counterweight to balance the robot when arm extends forward -->
+  <!-- Positioned at rear of robot to prevent forward tilting -->
+  <!-- Mass calculated to counteract arm (0.6kg at ~0.2m forward) with weight at ~0.22m rear -->
+  <xacro:property name="counterweight_mass" value="0.8" />  <!-- kg - adjustable -->
+  <joint name="$(arg prefix)counterweight_joint" type="fixed">
+    <parent link="$(arg prefix)base_link"/>
+    <child link="$(arg prefix)counterweight_link"/>
+    <!-- Position: rear of robot, low center of gravity -->
+    <!-- x=-0.22m puts it behind the rear casters (-0.177m) -->
+    <!-- z=0.02m keeps it low for stability -->
+    <origin xyz="-0.22 0.0 0.02" rpy="0 0 0"/>
+  </joint>
+  <link name="$(arg prefix)counterweight_link">
+    <visual>
+      <!-- Visual representation: compact weight block -->
+      <origin xyz="0 0 0" rpy="0 0 0"/>
+      <geometry>
+        <box size="0.06 0.12 0.04"/>  <!-- 6cm x 12cm x 4cm block -->
+      </geometry>
+      <material name="dark"/>
+    </visual>
+    <collision>
+      <origin xyz="0 0 0" rpy="0 0 0"/>
+      <geometry>
+        <box size="0.06 0.12 0.04"/>
+      </geometry>
+    </collision>
+    <inertial>
+      <origin xyz="0 0 0"/>
+      <mass value="${counterweight_mass}"/>
+      <!-- Inertia for solid box: I = (1/12) * m * (h^2 + d^2) etc. -->
+      <!-- For 0.8kg box of 0.06 x 0.12 x 0.04 m -->
+      <inertia ixx="${(1.0/12.0) * counterweight_mass * (0.12*0.12 + 0.04*0.04)}"
+               ixy="0.0" ixz="0.0"
+               iyy="${(1.0/12.0) * counterweight_mass * (0.06*0.06 + 0.04*0.04)}"
+               iyz="0.0"
+               izz="${(1.0/12.0) * counterweight_mass * (0.06*0.06 + 0.12*0.12)}"/>
+    </inertial>
+  </link>
   <xacro:turtlebot3_manipulation_system
     name="TurtleBot3ManipulationSystem" prefix="$(arg prefix)" use_sim="$(arg use_sim)"
